File: backplane.brd (EAGLE design)
At the start: 153.7 x 128.3 mm, 71 parts, among them J1 L717HDE15PD4CH4R, J10 5013310807, J11 5013310807, J12 5013310807, J13 5013310807, J14 5013311007, J15 5013311007, J16 5013311007, J17 5013311007, J18 5013311007, J19 5013311007, J2 1054301102, J20 5013311007, J21 5013311007, J22 5013311007, J23 5013311007, J24 SEAM-40-03.0-S-06-2-A-K-TR, J25 5055670271, J26 SAMTEC-TST-110-01-X-DJ, J27 SAMTEC-TST-110-01-X-DJ, J28 SAMTEC-TST-110-01-X-DJ, J29 SAMTEC-TST-110-01-X-DJ, J3 5011902017, J4 5013310807, J5 5013310807, J6 5013310807, J7 5013310807, J8 5013310807, J9 5013310807, U1 AM26LV32EIPWR, U10 AM26LV32EIPWR, U11 LP3962EMP-3.3, U2 AM26LV32EIPWR, U3 AM26LV32EIPWR, U4 AM26LV32EIPWR, U5 AM26LV32EIPWR, U6 AM26LV32EIPWR, U7 AM26LV32EIPWR, U8 AM26LV32EIPWR, U9 AM26LV32EIPWR

Commit message: Design Review Finished, Ready to order
Parts:
- C13: value (none) -> 0.1uF
Changed lines of the file:
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@@
 <hole x="3.2004" y="58.42" drill="3.3"/>
 <circle x="3.2004" y="58.42" radius="2.75" width="0.2" layer="48"/>
+<wire x1="33.7" y1="26.2" x2="35.6" y2="26.2" width="0.3048" layer="41"/>
 </plain>
 <attributes>
@@
 <attribute name="VALUE" x="62.065" y="102.075" size="1.27" layer="27" rot="R270"/>
 </element>
-<element name="C13" library="rcl" library_urn="urn:adsk.eagle:library:334" package="C0603" package3d_urn="urn:adsk.eagle:package:23616/2" value="" x="140.25" y="91.25" smashed="yes" rot="R180">
+<element name="C13" library="rcl" library_urn="urn:adsk.eagle:library:334" package="C0603" package3d_urn="urn:adsk.eagle:package:23616/2" value="0.1uF" x="140.25" y="91.25" smashed="yes" rot="R180">
 <attribute name="NAME" x="140.885" y="90.615" size="1.27" layer="25" rot="R180"/>
 <attribute name="POPULARITY" value="73" x="140.25" y="91.25" size="1.778" layer="27" rot="R180" display="off"/>
