File: backplane.sch (EAGLE design)
At the start: 71 parts, among them J1 L717HDE15PD4CH4R, J10 5013310807, J11 5013310807, J12 5013310807, J13 5013310807, J14 5013311007, J15 5013311007, J16 5013311007, J17 5013311007, J18 5013311007, J19 5013311007, J2 1054301102, J20 5013311007, J21 5013311007, J22 5013311007, J23 5013311007, J24 SEAM-40-03.0-S-06-2-A-K-TR, J25 5055670271, J26 SAMTEC-TST-110-01-X-DJ, J27 SAMTEC-TST-110-01-X-DJ, J28 SAMTEC-TST-110-01-X-DJ, J29 SAMTEC-TST-110-01-X-DJ, J3 5011902017, J4 5013310807, J5 5013310807, J6 5013310807, J7 5013310807, J8 5013310807, J9 5013310807, U1 AM26LV32EIPWR, U10 AM26LV32EIPWR, U11 LP3962EMP-3.3, U2 AM26LV32EIPWR, U3 AM26LV32EIPWR, U4 AM26LV32EIPWR, U5 AM26LV32EIPWR, U6 AM26LV32EIPWR, U7 AM26LV32EIPWR, U8 AM26LV32EIPWR, U9 AM26LV32EIPWR

Commit message: Design Review Finished, Ready to order
Parts:
- C13: value (none) -> 0.1uF
Changed lines of the file:
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@@
 <part name="GND44" library="supply1" library_urn="urn:adsk.eagle:library:371" deviceset="GND" device=""/>
 <part name="C11" library="rcl" library_urn="urn:adsk.eagle:library:334" deviceset="C-EU" device="C0603" package3d_urn="urn:adsk.eagle:package:23616/2" value="4.7uF"/>
-<part name="C13" library="rcl" library_urn="urn:adsk.eagle:library:334" deviceset="C-EU" device="C0603" package3d_urn="urn:adsk.eagle:package:23616/2"/>
+<part name="C13" library="rcl" library_urn="urn:adsk.eagle:library:334" deviceset="C-EU" device="C0603" package3d_urn="urn:adsk.eagle:package:23616/2" value="0.1uF"/>
 <part name="C12" library="sbrio_backplane" deviceset="875105144010" device=""/>
 <part name="L1" library="sbrio_backplane" deviceset="74437324068" device=""/>
